File: LED-Driver-CC.kicad_sch (KiCad schematic)
At the start: 7 parts, among them U5 TPS61165DBV

Commit message: Next iteration
Parts:
- renumbered C19 to C10, C20 to C11, C18 to C9, L3 to L1
Changed lines of the file:
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@@
 		(dnp no)
 		(fields_autoplaced yes)
-		(property "Reference" "#PWR039"
+		(property "Reference" "#PWR029"
 			(at 90.17 97.79 0)
 			(effects
@@
 		(instances
 			(project "prox_sensor"
+				(path "/72306bb1-8a24-469b-bdd7-d5938b058a41/c383466c-c754-4d27-b589-f85e884ef01b"
+					(reference "#PWR050")
+					(unit 1)
+				)
+				(path "/72306bb1-8a24-469b-bdd7-d5938b058a41/d998cc98-bbae-4acb-a979-e8a4326d62ac"
+					(reference "#PWR044")
+					(unit 1)
+				)
 				(path "/72306bb1-8a24-469b-bdd7-d5938b058a41/d99b5f2f-0228-47be-85b3-de9bfd376eab"
-					(reference "#PWR039")
+					(reference "#PWR029")
 					(unit 1)
 				)
@@
 		)
 		(instances
-			(project ""
+			(project "prox_sensor"
+				(path "/72306bb1-8a24-469b-bdd7-d5938b058a41/c383466c-c754-4d27-b589-f85e884ef01b"
+					(reference "D3")
+					(unit 1)
+				)
+				(path "/72306bb1-8a24-469b-bdd7-d5938b058a41/d998cc98-bbae-4acb-a979-e8a4326d62ac"
+					(reference "D2")
+					(unit 1)
+				)
 				(path "/72306bb1-8a24-469b-bdd7-d5938b058a41/d99b5f2f-0228-47be-85b3-de9bfd376eab"
 					(reference "D1")
@@
 		(dnp no)
 		(fields_autoplaced yes)
-		(property "Reference" "#PWR038"
+		(property "Reference" "#PWR031"
 			(at 130.81 127 0)
 			(effects
@@
 		(instances
 			(project "prox_sensor"
+				(path "/72306bb1-8a24-469b-bdd7-d5938b058a41/c383466c-c754-4d27-b589-f85e884ef01b"
+					(reference "#PWR052")
+					(unit 1)
+				)
+				(path "/72306bb1-8a24-469b-bdd7-d5938b058a41/d998cc98-bbae-4acb-a979-e8a4326d62ac"
+					(reference "#PWR046")
+					(unit 1)
+				)
 				(path "/72306bb1-8a24-469b-bdd7-d5938b058a41/d99b5f2f-0228-47be-85b3-de9bfd376eab"
-					(reference "#PWR038")
+					(reference "#PWR031")
 					(unit 1)
 				)
@@
 		(instances
 			(project "prox_sensor"
+				(path "/72306bb1-8a24-469b-bdd7-d5938b058a41/c383466c-c754-4d27-b589-f85e884ef01b"
+					(reference "R9")
+					(unit 1)
+				)
+				(path "/72306bb1-8a24-469b-bdd7-d5938b058a41/d998cc98-bbae-4acb-a979-e8a4326d62ac"
+					(reference "R8")
+					(unit 1)
+				)
 				(path "/72306bb1-8a24-469b-bdd7-d5938b058a41/d99b5f2f-0228-47be-85b3-de9bfd376eab"
 					(reference "R7")
@@
 		(dnp no)
 		(fields_autoplaced yes)
-		(property "Reference" "#PWR041"
+		(property "Reference" "#PWR030"
 			(at 110.49 127 0)
 			(effects
@@
 		(instances
 			(project "prox_sensor"
+				(path "/72306bb1-8a24-469b-bdd7-d5938b058a41/c383466c-c754-4d27-b589-f85e884ef01b"
+					(reference "#PWR051")
+					(unit 1)
+				)
+				(path "/72306bb1-8a24-469b-bdd7-d5938b058a41/d998cc98-bbae-4acb-a979-e8a4326d62ac"
+					(reference "#PWR045")
+					(unit 1)
+				)
 				(path "/72306bb1-8a24-469b-bdd7-d5938b058a41/d99b5f2f-0228-47be-85b3-de9bfd376eab"
-					(reference "#PWR041")
+					(reference "#PWR030")
 					(unit 1)
 				)
@@
 		(dnp no)
 		(fields_autoplaced yes)
-		(property "Reference" "#PWR040"
+		(property "Reference" "#PWR028"
 			(at 90.17 73.66 0)
 			(effects
@@
 		)
 		(instances
-			(project ""
+			(project "prox_sensor"
+				(path "/72306bb1-8a24-469b-bdd7-d5938b058a41/c383466c-c754-4d27-b589-f85e884ef01b"
+					(reference "#PWR049")
+					(unit 1)
+				)
+				(path "/72306bb1-8a24-469b-bdd7-d5938b058a41/d998cc98-bbae-4acb-a979-e8a4326d62ac"
+					(reference "#PWR043")
+					(unit 1)
+				)
 				(path "/72306bb1-8a24-469b-bdd7-d5938b058a41/d99b5f2f-0228-47be-85b3-de9bfd376eab"
-					(reference "#PWR040")
+					(reference "#PWR028")
 					(unit 1)
 				)
@@
 		(on_board yes)
 		(dnp no)
-		(property "Reference" "C20"
+		(property "Reference" "C11"
 			(at 178.816 89.154 90)
 			(effects
@@
 		(instances
 			(project "prox_sensor"
+				(path "/72306bb1-8a24-469b-bdd7-d5938b058a41/c383466c-c754-4d27-b589-f85e884ef01b"
+					(reference "C19")
+					(unit 1)
+				)
+				(path "/72306bb1-8a24-469b-bdd7-d5938b058a41/d998cc98-bbae-4acb-a979-e8a4326d62ac"
+					(reference "C16")
+					(unit 1)
+				)
 				(path "/72306bb1-8a24-469b-bdd7-d5938b058a41/d99b5f2f-0228-47be-85b3-de9bfd376eab"
-					(reference "C20")
+					(reference "C11")
 					(unit 1)
 				)
@@
 		(dnp no)
 		(fields_autoplaced yes)
-		(property "Reference" "#PWR043"
+		(property "Reference" "#PWR033"
 			(at 195.58 135.89 0)
 			(effects
@@
 		(instances
 			(project "prox_sensor"
+				(path "/72306bb1-8a24-469b-bdd7-d5938b058a41/c383466c-c754-4d27-b589-f85e884ef01b"
+					(reference "#PWR054")
+					(unit 1)
+				)
+				(path "/72306bb1-8a24-469b-bdd7-d5938b058a41/d998cc98-bbae-4acb-a979-e8a4326d62ac"
+					(reference "#PWR048")
+					(unit 1)
+				)
 				(path "/72306bb1-8a24-469b-bdd7-d5938b058a41/d99b5f2f-0228-47be-85b3-de9bfd376eab"
-					(reference "#PWR043")
+					(reference "#PWR033")
 					(unit 1)
 				)
@@
 		(on_board yes)
 		(dnp no)
-		(property "Reference" "L3"
+		(property "Reference" "L1"
 			(at 127 71.12 90)
 			(effects
@@
 		)
 		(instances
-			(project ""
+			(project "prox_sensor"
+				(path "/72306bb1-8a24-469b-bdd7-d5938b058a41/c383466c-c754-4d27-b589-f85e884ef01b"
+					(reference "L3")
+					(unit 1)
+				)
+				(path "/72306bb1-8a24-469b-bdd7-d5938b058a41/d998cc98-bbae-4acb-a979-e8a4326d62ac"
+					(reference "L2")
+					(unit 1)
+				)
 				(path "/72306bb1-8a24-469b-bdd7-d5938b058a41/d99b5f2f-0228-47be-85b3-de9bfd376eab"
-					(reference "L3")
+					(reference "L1")
 					(unit 1)
 				)
@@
 		(on_board yes)
 		(dnp no)
-		(property "Reference" "C18"
+		(property "Reference" "C9"
 			(at 91.948 91.186 90)
 			(effects
@@
 		(instances
 			(project "prox_sensor"
+				(path "/72306bb1-8a24-469b-bdd7-d5938b058a41/c383466c-c754-4d27-b589-f85e884ef01b"
+					(reference "C17")
+					(unit 1)
+				)
+				(path "/72306bb1-8a24-469b-bdd7-d5938b058a41/d998cc98-bbae-4acb-a979-e8a4326d62ac"
+					(reference "C14")
+					(unit 1)
+				)
 				(path "/72306bb1-8a24-469b-bdd7-d5938b058a41/d99b5f2f-0228-47be-85b3-de9bfd376eab"
-					(reference "C18")
+					(reference "C9")
 					(unit 1)
 				)
@@
 		)
 		(instances
-			(project ""
+			(project "prox_sensor"
+				(path "/72306bb1-8a24-469b-bdd7-d5938b058a41/c383466c-c754-4d27-b589-f85e884ef01b"
+					(reference "U8")
+					(unit 1)
+				)
+				(path "/72306bb1-8a24-469b-bdd7-d5938b058a41/d998cc98-bbae-4acb-a979-e8a4326d62ac"
+					(reference "U7")
+					(unit 1)
+				)
 				(path "/72306bb1-8a24-469b-bdd7-d5938b058a41/d99b5f2f-0228-47be-85b3-de9bfd376eab"
 					(reference "U5")
@@
 		(dnp no)
 		(fields_autoplaced yes)
-		(property "Reference" "#PWR042"
+		(property "Reference" "#PWR032"
 			(at 176.53 92.71 0)
 			(effects
@@
 		(instances
 			(project "prox_sensor"
+				(path "/72306bb1-8a24-469b-bdd7-d5938b058a41/c383466c-c754-4d27-b589-f85e884ef01b"
+					(reference "#PWR053")
+					(unit 1)
+				)
+				(path "/72306bb1-8a24-469b-bdd7-d5938b058a41/d998cc98-bbae-4acb-a979-e8a4326d62ac"
+					(reference "#PWR047")
+					(unit 1)
+				)
 				(path "/72306bb1-8a24-469b-bdd7-d5938b058a41/d99b5f2f-0228-47be-85b3-de9bfd376eab"
-					(reference "#PWR042")
+					(reference "#PWR032")
 					(unit 1)
 				)
@@
 		(on_board yes)
 		(dnp no)
-		(property "Reference" "C19"
+		(property "Reference" "C10"
 			(at 112.268 114.046 90)
 			(effects
@@
 		(instances
 			(project "prox_sensor"
+				(path "/72306bb1-8a24-469b-bdd7-d5938b058a41/c383466c-c754-4d27-b589-f85e884ef01b"
+					(reference "C18")
+					(unit 1)
+				)
+				(path "/72306bb1-8a24-469b-bdd7-d5938b058a41/d998cc98-bbae-4acb-a979-e8a4326d62ac"
+					(reference "C15")
+					(unit 1)
+				)
 				(path "/72306bb1-8a24-469b-bdd7-d5938b058a41/d99b5f2f-0228-47be-85b3-de9bfd376eab"
-					(reference "C19")
-					(unit 1)
-				)
+					(reference "C10")
+					(unit 1)
+				)
