File: LED-Driver-CC.kicad_sch (KiCad schematic)
At the start: 7 parts, among them U5 TPS61165DBV

Commit message: Adding power control and extra input, to attach another som
Parts:
- D1: LCSC Part # (none) -> C116159
- L3: LCSC Part # (none) -> C2858406
- U5: LCSC Part # (none) -> C58756
Changed lines of the file:
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@@
+			)
+		)
+		(property "LCSC Part #" "C116159"
+			(at 152.4 76.2 0)
+			(effects
+				(font
+					(size 1.27 1.27)
+				)
+				(hide yes)
 			)
 		)
@@
 			)
 		)
+		(property "LCSC Part #" "C2858406"
+			(at 127 76.2 90)
+			(effects
+				(font
+					(size 1.27 1.27)
+				)
+				(hide yes)
+			)
+		)
 		(pin "2"
 		)
@@
 			(at 130.81 97.79 0)
 			(effects
+				(font
+					(size 1.27 1.27)
+				)
+				(hide yes)
+			)
+		)
+		(property "LCSC Part #" "C58756"
+			(at 130.81 97.79 0)
+			(effects
