File: STHS34PF80TR.kicad_sch (KiCad schematic)
At the start: 2 parts, among them U3 STHS34PF80

Commit message: Next iteration
Parts:
- renumbered C25 to C12, U3 to U6
Changed lines of the file:
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@@
 		(dnp no)
 		(fields_autoplaced yes)
-		(property "Reference" "U3"
+		(property "Reference" "U6"
 			(at 162.56 109.1498 0)
 			(effects
@@
 			(project ""
 				(path "/72306bb1-8a24-469b-bdd7-d5938b058a41/c7a69e2a-1737-423f-8ec2-47bf6b5b87b3"
-					(reference "U3")
+					(reference "U6")
 					(unit 1)
 				)
@@
 		(dnp no)
 		(fields_autoplaced yes)
-		(property "Reference" "#PWR055"
+		(property "Reference" "#PWR035"
 			(at 105.41 111.76 0)
 			(effects
@@
 			(project "prox_sensor"
 				(path "/72306bb1-8a24-469b-bdd7-d5938b058a41/c7a69e2a-1737-423f-8ec2-47bf6b5b87b3"
-					(reference "#PWR055")
+					(reference "#PWR035")
 					(unit 1)
 				)
@@
 		(on_board yes)
 		(dnp no)
-		(property "Reference" "C25"
+		(property "Reference" "C12"
 			(at 158.496 83.312 0)
 			(effects
@@
 			(project "prox_sensor"
 				(path "/72306bb1-8a24-469b-bdd7-d5938b058a41/c7a69e2a-1737-423f-8ec2-47bf6b5b87b3"
-					(reference "C25")
+					(reference "C12")
 					(unit 1)
 				)
@@
 		(dnp no)
 		(fields_autoplaced yes)
-		(property "Reference" "#PWR052"
+		(property "Reference" "#PWR038"
 			(at 154.94 95.25 0)
 			(effects
@@
 			(project "prox_sensor"
 				(path "/72306bb1-8a24-469b-bdd7-d5938b058a41/c7a69e2a-1737-423f-8ec2-47bf6b5b87b3"
-					(reference "#PWR052")
+					(reference "#PWR038")
 					(unit 1)
 				)
@@
 		(on_board yes)
 		(dnp no)
-		(property "Reference" "#PWR054"
+		(property "Reference" "#PWR034"
 			(at 102.87 80.01 0)
 			(effects
@@
 			(project "prox_sensor"
 				(path "/72306bb1-8a24-469b-bdd7-d5938b058a41/c7a69e2a-1737-423f-8ec2-47bf6b5b87b3"
-					(reference "#PWR054")
+					(reference "#PWR034")
 					(unit 1)
 				)
@@
 		(dnp no)
 		(fields_autoplaced yes)
-		(property "Reference" "#PWR053"
+		(property "Reference" "#PWR037"
 			(at 147.32 135.89 0)
 			(effects
@@
 			(project "prox_sensor"
 				(path "/72306bb1-8a24-469b-bdd7-d5938b058a41/c7a69e2a-1737-423f-8ec2-47bf6b5b87b3"
-					(reference "#PWR053")
+					(reference "#PWR037")
 					(unit 1)
 				)
@@
 		(on_board yes)
 		(dnp no)
-		(property "Reference" "#PWR051"
+		(property "Reference" "#PWR036"
 			(at 147.32 80.01 0)
 			(effects
@@
 			(project "prox_sensor"
 				(path "/72306bb1-8a24-469b-bdd7-d5938b058a41/c7a69e2a-1737-423f-8ec2-47bf6b5b87b3"
-					(reference "#PWR051")
-					(unit 1)
-				)
+					(reference "#PWR036")
+					(unit 1)
+				)
