File: STM32.kicad_sch (KiCad schematic)
At the start: 6 parts, among them J12 Conn_01x05, U2 STM32L031G6U6

Commit message: Next iteration
Parts:
- renumbered C2 to C4, C7 to C5, C8 to C6, J12 to J7, R4 to R6, U2 to U3
Changed lines of the file:
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@@
 		(on_board yes)
 		(dnp no)
-		(property "Reference" "C2"
+		(property "Reference" "C4"
 			(at 86.614 107.442 0)
 			(effects
@@
 			(project "prox_sensor"
 				(path "/72306bb1-8a24-469b-bdd7-d5938b058a41/03ce4162-687c-4e63-8ec8-c46aac94fbf4"
-					(reference "C2")
+					(reference "C4")
 					(unit 1)
 				)
@@
 		(dnp no)
 		(fields_autoplaced yes)
-		(property "Reference" "#PWR018"
+		(property "Reference" "#PWR020"
 			(at 137.16 96.52 0)
 			(effects
@@
 			(project "prox_sensor"
 				(path "/72306bb1-8a24-469b-bdd7-d5938b058a41/03ce4162-687c-4e63-8ec8-c46aac94fbf4"
-					(reference "#PWR018")
+					(reference "#PWR020")
 					(unit 1)
 				)
@@
 		(on_board yes)
 		(dnp no)
-		(property "Reference" "C8"
+		(property "Reference" "C6"
 			(at 147.574 88.138 90)
 			(effects
@@
 			(project "prox_sensor"
 				(path "/72306bb1-8a24-469b-bdd7-d5938b058a41/03ce4162-687c-4e63-8ec8-c46aac94fbf4"
-					(reference "C8")
+					(reference "C6")
 					(unit 1)
 				)
@@
 		(on_board yes)
 		(dnp no)
-		(property "Reference" "U2"
+		(property "Reference" "U3"
 			(at 163.068 143.764 0)
 			(effects
@@
 			(project "prox_sensor"
 				(path "/72306bb1-8a24-469b-bdd7-d5938b058a41/03ce4162-687c-4e63-8ec8-c46aac94fbf4"
-					(reference "U2")
+					(reference "U3")
 					(unit 1)
 				)
@@
 		(on_board yes)
 		(dnp no)
-		(property "Reference" "C7"
+		(property "Reference" "C5"
 			(at 138.938 91.186 90)
 			(effects
@@
 			(project "prox_sensor"
 				(path "/72306bb1-8a24-469b-bdd7-d5938b058a41/03ce4162-687c-4e63-8ec8-c46aac94fbf4"
-					(reference "C7")
+					(reference "C5")
 					(unit 1)
 				)
@@
 		(on_board yes)
 		(dnp no)
-		(property "Reference" "#PWR05"
+		(property "Reference" "#PWR016"
 			(at 54.61 73.66 0)
 			(effects
@@
 			(project "prox_sensor"
 				(path "/72306bb1-8a24-469b-bdd7-d5938b058a41/03ce4162-687c-4e63-8ec8-c46aac94fbf4"
-					(reference "#PWR05")
+					(reference "#PWR016")
 					(unit 1)
 				)
@@
 		(dnp no)
 		(fields_autoplaced yes)
-		(property "Reference" "#PWR014"
+		(property "Reference" "#PWR021"
 			(at 146.05 96.52 0)
 			(effects
@@
 			(project "prox_sensor"
 				(path "/72306bb1-8a24-469b-bdd7-d5938b058a41/03ce4162-687c-4e63-8ec8-c46aac94fbf4"
-					(reference "#PWR014")
+					(reference "#PWR021")
 					(unit 1)
 				)
@@
 		(dnp no)
 		(fields_autoplaced yes)
-		(property "Reference" "#PWR017"
+		(property "Reference" "#PWR023"
 			(at 154.94 151.13 0)
 			(effects
@@
 			(project "prox_sensor"
 				(path "/72306bb1-8a24-469b-bdd7-d5938b058a41/03ce4162-687c-4e63-8ec8-c46aac94fbf4"
-					(reference "#PWR017")
+					(reference "#PWR023")
 					(unit 1)
 				)
@@
 		(dnp no)
 		(fields_autoplaced yes)
-		(property "Reference" "#PWR08"
+		(property "Reference" "#PWR018"
 			(at 90.17 123.19 0)
 			(effects
@@
 			(project "prox_sensor"
 				(path "/72306bb1-8a24-469b-bdd7-d5938b058a41/03ce4162-687c-4e63-8ec8-c46aac94fbf4"
-					(reference "#PWR08")
+					(reference "#PWR018")
 					(unit 1)
 				)
@@
 		(on_board yes)
 		(dnp no)
-		(property "Reference" "R4"
+		(property "Reference" "R6"
 			(at 102.616 115.57 90)
 			(effects
@@
 			(project "prox_sensor"
 				(path "/72306bb1-8a24-469b-bdd7-d5938b058a41/03ce4162-687c-4e63-8ec8-c46aac94fbf4"
-					(reference "R4")
+					(reference "R6")
 					(unit 1)
 				)
@@
 		(dnp no)
 		(fields_autoplaced yes)
-		(property "Reference" "#PWR09"
+		(property "Reference" "#PWR019"
 			(at 95.25 123.19 0)
 			(effects
@@
 			(project "prox_sensor"
 				(path "/72306bb1-8a24-469b-bdd7-d5938b058a41/03ce4162-687c-4e63-8ec8-c46aac94fbf4"
-					(reference "#PWR09")
+					(reference "#PWR019")
 					(unit 1)
 				)
@@
 		(on_board yes)
 		(dnp no)
-		(property "Reference" "#PWR016"
+		(property "Reference" "#PWR022"
 			(at 152.4 74.93 0)
 			(effects
@@
 			(project "prox_sensor"
 				(path "/72306bb1-8a24-469b-bdd7-d5938b058a41/03ce4162-687c-4e63-8ec8-c46aac94fbf4"
-					(reference "#PWR016")
+					(reference "#PWR022")
 					(unit 1)
 				)
@@
 		(dnp no)
 		(fields_autoplaced yes)
-		(property "Reference" "J12"
+		(property "Reference" "J7"
 			(at 85.09 77.4699 0)
 			(effects
@@
 			(project ""
 				(path "/72306bb1-8a24-469b-bdd7-d5938b058a41/03ce4162-687c-4e63-8ec8-c46aac94fbf4"
-					(reference "J12")
+					(reference "J7")
 					(unit 1)
 				)
@@
 		(dnp no)
 		(fields_autoplaced yes)
-		(property "Reference" "#PWR01"
+		(property "Reference" "#PWR017"
 			(at 44.45 83.82 0)
 			(effects
@@
 			(project "prox_sensor"
 				(path "/72306bb1-8a24-469b-bdd7-d5938b058a41/03ce4162-687c-4e63-8ec8-c46aac94fbf4"
-					(reference "#PWR01")
+					(reference "#PWR017")
 					(unit 1)
 				)
