File: ToF.kicad_sch (KiCad schematic)
At the start: 3 parts, among them U4 VL53L0CXV0DH1

Commit message: Next iteration
Parts:
- renumbered C13 to C7, C16 to C8
Changed lines of the file:
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@@
 		(on_board yes)
 		(dnp no)
-		(property "Reference" "C16"
+		(property "Reference" "C8"
 			(at 159.004 74.168 90)
 			(effects
@@
 			(project "prox_sensor"
 				(path "/72306bb1-8a24-469b-bdd7-d5938b058a41/61bea680-b05a-452c-a186-15fdfa8712c0"
-					(reference "C16")
+					(reference "C8")
 					(unit 1)
 				)
@@
 		(on_board yes)
 		(dnp no)
-		(property "Reference" "C13"
+		(property "Reference" "C7"
 			(at 150.368 77.216 90)
 			(effects
@@
 			(project "prox_sensor"
 				(path "/72306bb1-8a24-469b-bdd7-d5938b058a41/61bea680-b05a-452c-a186-15fdfa8712c0"
-					(reference "C13")
+					(reference "C7")
 					(unit 1)
 				)
@@
 		(on_board yes)
 		(dnp no)
-		(property "Reference" "#PWR021"
+		(property "Reference" "#PWR027"
 			(at 187.96 63.5 0)
 			(effects
@@
 			(project "prox_sensor"
 				(path "/72306bb1-8a24-469b-bdd7-d5938b058a41/61bea680-b05a-452c-a186-15fdfa8712c0"
-					(reference "#PWR021")
+					(reference "#PWR027")
 					(unit 1)
 				)
@@
 		(dnp no)
 		(fields_autoplaced yes)
-		(property "Reference" "#PWR034"
+		(property "Reference" "#PWR026"
 			(at 157.48 82.55 0)
 			(effects
@@
 			(project "prox_sensor"
 				(path "/72306bb1-8a24-469b-bdd7-d5938b058a41/61bea680-b05a-452c-a186-15fdfa8712c0"
-					(reference "#PWR034")
+					(reference "#PWR026")
 					(unit 1)
 				)
@@
 		(dnp no)
 		(fields_autoplaced yes)
-		(property "Reference" "#PWR026"
+		(property "Reference" "#PWR025"
 			(at 148.59 82.55 0)
 			(effects
@@
 			(project "prox_sensor"
 				(path "/72306bb1-8a24-469b-bdd7-d5938b058a41/61bea680-b05a-452c-a186-15fdfa8712c0"
-					(reference "#PWR026")
+					(reference "#PWR025")
 					(unit 1)
 				)
@@
 		(dnp no)
 		(fields_autoplaced yes)
-		(property "Reference" "#PWR020"
+		(property "Reference" "#PWR024"
 			(at 138.43 119.38 0)
 			(effects
@@
 			(project "prox_sensor"
 				(path "/72306bb1-8a24-469b-bdd7-d5938b058a41/61bea680-b05a-452c-a186-15fdfa8712c0"
-					(reference "#PWR020")
+					(reference "#PWR024")
 					(unit 1)
 				)
