File: VEML7700-TR.kicad_sch (KiCad schematic)
At the start: 2 parts

Commit message: Next iteration
Parts:
- renumbered C26 to C13
Changed lines of the file:
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@@
 		(on_board yes)
 		(dnp no)
-		(property "Reference" "#PWR058"
+		(property "Reference" "#PWR041"
 			(at 137.16 81.28 0)
 			(effects
@@
 			(project "prox_sensor"
 				(path "/72306bb1-8a24-469b-bdd7-d5938b058a41/7a84920f-36d6-4cc4-99b6-ae3fc4d300dd"
-					(reference "#PWR058")
+					(reference "#PWR041")
 					(unit 1)
 				)
@@
 		(on_board yes)
 		(dnp no)
-		(property "Reference" "#PWR060"
+		(property "Reference" "#PWR039"
 			(at 119.38 90.17 0)
 			(effects
@@
 			(project "prox_sensor"
 				(path "/72306bb1-8a24-469b-bdd7-d5938b058a41/7a84920f-36d6-4cc4-99b6-ae3fc4d300dd"
-					(reference "#PWR060")
+					(reference "#PWR039")
 					(unit 1)
 				)
@@
 		(on_board yes)
 		(dnp no)
-		(property "Reference" "C26"
+		(property "Reference" "C13"
 			(at 122.936 93.472 0)
 			(effects
@@
 			(project "prox_sensor"
 				(path "/72306bb1-8a24-469b-bdd7-d5938b058a41/7a84920f-36d6-4cc4-99b6-ae3fc4d300dd"
-					(reference "C26")
+					(reference "C13")
 					(unit 1)
 				)
@@
 		(dnp no)
 		(fields_autoplaced yes)
-		(property "Reference" "#PWR061"
+		(property "Reference" "#PWR040"
 			(at 119.38 107.95 0)
 			(effects
@@
 			(project "prox_sensor"
 				(path "/72306bb1-8a24-469b-bdd7-d5938b058a41/7a84920f-36d6-4cc4-99b6-ae3fc4d300dd"
-					(reference "#PWR061")
+					(reference "#PWR040")
 					(unit 1)
 				)
@@
 		(dnp no)
 		(fields_autoplaced yes)
-		(property "Reference" "#PWR059"
+		(property "Reference" "#PWR042"
 			(at 127 83.82 0)
 			(effects
@@
 			(project "prox_sensor"
 				(path "/72306bb1-8a24-469b-bdd7-d5938b058a41/7a84920f-36d6-4cc4-99b6-ae3fc4d300dd"
-					(reference "#PWR059")
+					(reference "#PWR042")
 					(unit 1)
 				)
