File: prox_sensor.kicad_pcb (KiCad board)
At the start: 4 copper layers, 25.1 x 45.3 mm, 37 parts, among them J1 +, J12 Conn_01x05, J2 -, J3 A, J9 K, U1 BD4840G-TR, U2 STM32L031G6U6, U3 STHS34PF80, U4 VL53L0CXV0DH1, U5 TPS61165DBV, U6 NCP718xSN330

Commit message: Next iteration
Parts:
- added C14: 4.7uF/10V, Capacitor_SMD:C_0402_1005Metric, B.Cu at (136.1, 146.2)
- added C15: 220nF/16V, Capacitor_SMD:C_0402_1005Metric, B.Cu at (132.6, 141.9)
- added C16: 1uF/25V, Capacitor_SMD:C_0402_1005Metric, B.Cu at (134.1, 152.8)
- added C17: 4.7uF/10V, Capacitor_SMD:C_0402_1005Metric, B.Cu at (135.8, 132.3)
- added C18: 220nF/16V, Capacitor_SMD:C_0402_1005Metric, B.Cu at (132.4, 127.7)
- added C19: 1uF/25V, Capacitor_SMD:C_0402_1005Metric, B.Cu at (133.7, 138.1)
- added D2: MBR0540, Diode_SMD:D_SOD-123, B.Cu at (133.1, 150.4)
- added D3: MBR0540, Diode_SMD:D_SOD-123, B.Cu at (132.9, 136.0)
- added J3: A, TestPoint:TestPoint_Pad_D2.0mm, B.Cu at (138.8, 155.5)
- added J4: K, TestPoint:TestPoint_Pad_D2.0mm, B.Cu at (138.8, 149.9)
- added J8: A, TestPoint:TestPoint_Pad_D2.0mm, B.Cu at (138.6, 141.0)
- added J9: K, TestPoint:TestPoint_Pad_D2.0mm, B.Cu at (138.6, 134.9)
- added L2: 10uH/0.5A, 1-COB-MOD:L_Murata_DFE201610P, B.Cu at (133.0, 148.0)
- added L3: 10uH/0.5A, 1-COB-MOD:L_Murata_DFE201610P, B.Cu at (132.7, 133.6)
- added R8: 1.3R, Capacitor_SMD:C_0603_1608Metric, B.Cu at (137.0, 152.5)
- added R9: 1.3R, Capacitor_SMD:C_0603_1608Metric, B.Cu at (136.7, 137.8)
- added U7: TPS61165DBV, Package_TO_SOT_SMD:SOT-23-6, B.Cu at (133.1, 144.6)
- added U8: TPS61165DBV, Package_TO_SOT_SMD:SOT-23-6, B.Cu at (132.8, 130.4)
- renumbered C24 to C1, C19 to C10, C20 to C11, C25 to C12, C26 to C13, C22 to C2, C23 to C3, C2 to C4, C7 to C5, C8 to C6, C13 to C7, C16 to C8, C18 to C9, J3 to J5, J9 to J6, J12 to J7, L3 to L1, R18 to R2, R20 to R3, R2 to R4, R3 to R5, R4 to R6, U6 to U2, U2 to U3, U3 to U6
Connections:
- net /TPS61165/LEDA renamed /TPS61165_R/LEDA
- net /TPS61165/LEDK renamed /TPS61165_R/LEDK
Routing:
- net /TPS61165_B/LEDK: track 0.00 -> 10.1 mm
- net /TPS61165_G/LEDK: track 0.00 -> 9.69 mm
- net Net-(U7-COMP): track 0.00 -> 1.62 mm
- net Net-(U8-COMP): track 0.00 -> 1.60 mm
- net GND: vias 77 -> 80
- net +BATT: vias 5 -> 20
- added copper zone on F.Cu, net +BATT
- added copper zone on B.Cu, net /TPS61165_B/LEDA
- added copper zone on B.Cu, net /TPS61165_B/LEDK
- added copper zone on B.Cu, net /TPS61165_G/LEDA
- added copper zone on B.Cu, net /TPS61165_G/LEDK
- added copper zone on B.Cu, net Net-(D2-A)
- added copper zone on B.Cu, net Net-(D3-A)
Other:
- board size 25.1 x 45.3 mm -> 29.9 x 49.9 mm
