File: prox_sensor.kicad_sch (KiCad schematic)
At the start: 17 parts, among them J1 +, J11 -, J2 -, J3 A, J4 -, J9 K, U1 BD4840G-TR, U6 NCP718xSN330

Commit message: Adding light sensor
Parts:
- renumbered J11 to GND1, J4 to VBUS1
Other:
- added sheet VEML7700-TR (VEML7700-TR.kicad_sch)

Commit message: Next iteration
Parts:
- added J3, J8: A, TestPoint:TestPoint_Pad_D2.0mm, symbol Connector_Generic:Conn_01x01
- added J4, J9: K, TestPoint:TestPoint_Pad_D2.0mm, symbol Connector_Generic:Conn_01x01
- renumbered C24 to C1, C22 to C2, C23 to C3, J3 to J5, J9 to J6, R18 to R2, R20 to R3, R2 to R4, R3 to R5, U6 to U2
Connections:
- new net TPS61165_B/LEDA: J8.1 (Pin_1)
- new net TPS61165_B/LEDK: J9.1 (Pin_1)
- new net TPS61165_G/LEDA: J3.1 (Pin_1)
- new net TPS61165_G/LEDK: J4.1 (Pin_1)
Other:
- sheet TPS61165 renamed TPS61165_R
- added sheet TPS61165_B (LED-Driver-CC.kicad_sch)
- added sheet TPS61165_G (LED-Driver-CC.kicad_sch)
